Commit message: Sit rail on bench top, spanning the full long edge; arms face across
- URDF: lengthen rail_base to 1.25 m and bake world_to_rail_base to place the
  rail on the bench top (z=0.30), centred on the long (X) edge end-to-end
- URDF: yaw both arm mounts -90 and offset them +/-90 mm along X so the arms
  sit side by side and reach across the bench toward -Y
- rail_joint travel 0.63 -> 1.10 m; teleop RAIL_MAX matched
- lab_scene: drop runtime place_robot_on_bench (placement now baked in URDF,
  robust vs fix_base); respread glassware along X within reach
- guide updated

Fixes rail sinking below the table and the short cross-wise rail.

File: model/omx_f_dual_on_rail.urdf (robot description, URDF)
Before this commit: robot omx_f_dual_on_rail, 21 links, 20 joints
Links:
- link rail_base: mass 3.0 -> 4.0; geometry collision box size=1.250 0.080 0.040; visual box size=1.250 0.080 0.040
- link rail_cart: geometry collision box size=0.300 0.140 0.060; visual box size=0.300 0.140 0.060
Joints:
- joint l_arm_mount: origin xyz=0 0.075 0.060 rpy=0 0 0 -> xyz=0.09 0 0.060 rpy=0 0 -1.5707963
- joint r_arm_mount: origin xyz=0 -0.075 0.060 rpy=0 0 0 -> xyz=-0.09 0 0.060 rpy=0 0 -1.5707963
- joint rail_joint: limit lower=0 upper=0.630 effort=100 velocity=0.5 -> lower=0 upper=1.100 effort=100 velocity=0.5
- joint world_to_rail_base: origin xyz=0 0 0 rpy=0 0 0 -> xyz=-0.625 0.30 0.30 rpy=0 0 0
